Commit message: Correctly scaled schunk model, added motion planning with quaternions

File: schunk_gripper_communication/urdf/lwa4p/lwa4p.urdf.xacro (robot description, xacro)
@@ -34,19 +34,19 @@
     <link name="camera_link">
       <inertial>
-        <origin xyz="0 0 0" rpy="0 0 0" />
+        <origin xyz="0 0 -0.13" rpy="0 0 0" />
         <mass value="10"/>
         <inertia ixx="0.01" ixy="0" ixz="0" iyy="0.01" iyz="0" izz="0.01" />
       </inertial>
        <visual>
-        <origin xyz="0 0 -0.01" rpy="1.57 0 0" />
-        <geometry>
-          <mesh filename="package://schunk_gripper_communication/meshes/cylinder-notop.dae" scale="1.85 0.2 1.85"/>
+        <origin xyz="0 0 -0.13" rpy="1.57 0 0" />
+        <geometry>
+          <mesh filename="package://schunk_gripper_communication/meshes/cylinder-notop.dae" scale="1.25 0.2 1.25"/>
         </geometry>
         <material name="Schunk/Yellow" />
       </visual>
       <collision>
-        <origin xyz="0 0 -0.01" rpy="1.57 0 0" />
-        <geometry>
-          <mesh filename="package://schunk_gripper_communication/meshes/cylinder-notop.dae" scale="1.85 0.2 1.85"/>
+        <origin xyz="0 0 -0.13" rpy="1.57 0 0" />
+        <geometry>
+          <mesh filename="package://schunk_gripper_communication/meshes/cylinder-notop.dae" scale="1.25 0.2 1.25"/>
         </geometry>
       </collision>
@@ -54,19 +54,19 @@
     <link name="table_link">
       <inertial>
-        <origin xyz="0 0 0" rpy="0 0 0" />
+        <origin xyz="0 0 -0.13" rpy="0 0 0" />
         <mass value="10"/>
         <inertia ixx="0.01" ixy="0" ixz="0" iyy="0.01" iyz="0" izz="0.01" />
       </inertial>
        <visual>
-        <origin xyz="0 0 0" rpy="0 0 0" />
-        <geometry>
-            <cylinder length="0.01" radius="0.9" />
+        <origin xyz="0 0 -0.13" rpy="0 0 0" />
+        <geometry>
+            <cylinder length="0.01" radius="0.61" />
         </geometry>
         <material name="Schunk/Yellow" />
       </visual>
       <collision>
-        <origin xyz="0 0 0" rpy="0 0 0" />
-        <geometry>
-            <cylinder length="0.01" radius="0.9" />
+        <origin xyz="0 0 -0.13" rpy="0 0 0" />
+        <geometry>
+            <cylinder length="0.01" radius="0.61" />
         </geometry>
       </collision>
@@ -291,6 +291,6 @@
     </link>
     -->
-    <joint name="gripper_joint" type="fixed" >
-        <origin xyz="0 0 0.27" rpy="0 0 0" />
+<joint name="gripper_joint" type="fixed" >
+        <origin xyz="0 0 0.29" rpy="0 0 0" />
         <parent link="${name}_6_link" />
       <child link="gripper_link" />
@@ -298,25 +298,25 @@
     <link name="gripper_link">
       <inertial>
-        <origin xyz="0 0 0.13" rpy="0 0 0" />
+        <origin xyz="0 0 0" rpy="0 0 0" />
         <mass value="0.5"/>
         <inertia ixx="0.01" ixy="0" ixz="0" iyy="0.01" iyz="0" izz="0.01" />
       </inertial>
        <visual>
-        <origin xyz="0 0 -0.15" rpy="0 0 0" />
-        <geometry>
-            <box size="0.1 0.1 0.10" />
+        <origin xyz="0 0 -0.11" rpy="0 0 0" />
+        <geometry>
+            <box size="0.1 0.1 0.227" />
         </geometry>
         <material name="Schunk/Yellow" />
       </visual>
       <collision>
-        <origin xyz="0 0 -0.15" rpy="0 0 0" />
-        <geometry>
-            <box size="0.1 0.1 0.10" />
-        </geometry>
-      </collision>
-     </link>
+        <origin xyz="0 0 -0.11" rpy="0 0 0" />
+        <geometry>
+            <box size="0.1 0.1 0.227" />
+        </geometry>
+      </collision>
+    </link>
 <!-- joint between arm_6_link and tcp_link -->
     <joint name="${name}_tcp_joint" type="fixed">
-      <origin xyz="0 0 0.08" rpy="0 0 0" />
+      <origin xyz="0 0 0.0" rpy="0 0 0" />
       <parent link="gripper_link"/>
       <child link="${name}_tcp_link"/>

Commit message: Added schunk launch file to agree wtih physical arm

File: schunk_gripper_communication/urdf/lwa4p/lwa4p.urdf.xacro (robot description, xacro)
@@ -303,14 +303,14 @@
       </inertial>
        <visual>
-        <origin xyz="0 0 -0.11" rpy="0 0 0" />
-        <geometry>
-            <box size="0.1 0.1 0.227" />
+        <origin xyz="0 0 -0.105" rpy="0 0 0" />
+        <geometry>
+            <box size="0.1 0.05 0.21" />
         </geometry>
         <material name="Schunk/Yellow" />
       </visual>
       <collision>
-        <origin xyz="0 0 -0.11" rpy="0 0 0" />
-        <geometry>
-            <box size="0.1 0.1 0.227" />
+        <origin xyz="0 0 -0.105" rpy="0 0 0" />
+        <geometry>
+            <box size="0.1 0.05 0.21" />
         </geometry>
       </collision>

Commit message: Reverted to older version

File: schunk_gripper_communication/urdf/lwa4p/lwa4p.urdf.xacro (robot description, xacro)
@@ -303,14 +303,14 @@
       </inertial>
        <visual>
-        <origin xyz="0 0 -0.105" rpy="0 0 0" />
-        <geometry>
-            <box size="0.1 0.05 0.21" />
+        <origin xyz="0 0 -0.11" rpy="0 0 0" />
+        <geometry>
+            <box size="0.1 0.1 0.227" />
         </geometry>
         <material name="Schunk/Yellow" />
       </visual>
       <collision>
-        <origin xyz="0 0 -0.105" rpy="0 0 0" />
-        <geometry>
-            <box size="0.1 0.05 0.21" />
+        <origin xyz="0 0 -0.11" rpy="0 0 0" />
+        <geometry>
+            <box size="0.1 0.1 0.227" />
         </geometry>
       </collision>
